Commit message: urtf files

File: week1/urdf/puzzle.urdf (robot description, URDF)
Before this commit: robot link_example, 4 links, 3 joints
Links:
- removed link link1
- removed link link2
- removed link link3
- removed link link4
- added link base_footprint
- added link base_link; visual mesh filename=package://week1/meshes/MCR2_puzzlebot_jetson_lidar_base.stl
- added link camera_base_link
- added link caster_holder_link; visual mesh filename=package://week1/meshes/MCR2_caster_wheel.stl
- added link lidar_base_link
- added link wheel_left_link; visual mesh filename=package://week1/meshes/MCR2_wheel.stl
- added link wheel_right_link; visual mesh filename=package://week1/meshes/MCR2_wheel.stl
Joints:
- removed joint joint1
- removed joint joint2
- removed joint joint3
- added joint base_link_joint: type fixed, parent base_footprint, child base_link, origin xyz=0 0 0.05 rpy=0 0 0
- added joint camera_base_joint: type fixed, parent base_link, child camera_base_link, origin xyz=0.112 0 0.065 rpy=0 0 0
- added joint caster_holder_joint: type fixed, parent base_link, child caster_holder_link, origin xyz=-0.095 0 -0.0307 rpy=0 0 0
- added joint lidar_base_joint: type fixed, parent base_link, child lidar_base_link, origin xyz=0.05 0 0.110 rpy=0 0 0
- added joint wheel_left_joint: type continuous, parent base_link, child wheel_left_link, origin xyz=0.052 0.095 -0.0025 rpy=0 0 0, axis 0 1 0
- added joint wheel_right_joint: type continuous, parent base_link, child wheel_right_link, origin xyz=0.052 -0.095 -0.0025 rpy=0 0 0, axis 0 1 0
