Commit message: Se agrega propuesta challenge2

File: challenge2/urdf/puzzle_mesh.urdf (robot description, URDF)
Before this commit: robot Puzzlebot_Jetson_Lidar_Ed., 7 links, 6 joints
Links:
- link wheel_left_link: geometry visual mesh filename=package://challenge1/meshes/MCR2_wheel.stl

Commit message: Se corrigue exportacion de archivos

File: challenge2/urdf/puzzle_mesh.urdf (robot description, URDF)
Before this commit: robot Puzzlebot_Jetson_Lidar_Ed., 7 links, 6 joints
Links:
- link base_link: geometry visual mesh filename=package://challenge2/meshes/MCR2_puzzlebot_jetson_lidar_bas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
- link caster_holder_link: geometry visual mesh filename=package://challenge2/meshes/MCR2_caster_wheel.stl
- link wheel_left_link: geometry visual mesh filename=package://challenge2/meshes/MCR2_wheel.stl
- link wheel_right_link: geometry visual mesh filename=package://challenge2/meshes/MCR2_wheel.stl
